Commit message: ready for estimator tuning

File: rosplane_sim/xacro/fixedwing.xacro (robot description, xacro)
@@ -7,5 +7,5 @@
   <xacro:property name="mesh_file" value="package://rosplane_sim/xacro/meshes/fixedwing.dae"/>
   <xacro:property name="body_width" value="1.54"/>
-  <xacro:property name="body_height" value="0.77" />
+  <xacro:property name="body_height" value="0.77"/>
   <xacro:property name="body_length" value="0.20"/>
   <xacro:property name="mass" value="1.5"/>
@@ -16,84 +16,62 @@
   <!-- Property Blocks -->
   <xacro:property name="empty_inertia">
-    <inertia ixx="0.0001" ixy="0.0" ixz="0.0" iyy="0.0001" iyz="0.0" izz="0.001" />
+    <inertia ixx="0.0001" ixy="0.0" ixz="0.0" iyy="0.0001" iyz="0.0" izz="0.001"/>
   </xacro:property>
   <!-- Instantiate Link and Visual -->
   <link name="${namespace}/base_link">
     <inertial>
-      <mass value="${mass}" />
-      <origin xyz="0 0 0" />
-      <inertia ixx="${Jx}" ixy="0.00" ixz="${Jxz}" iyy="${Jy}" iyz="0.00" izz="${Jz}" />
+      <mass value="${mass}"/>
+      <origin xyz="0 0 0"/>
+      <inertia ixx="${Jx}" ixy="0.00" ixz="${Jxz}" iyy="${Jy}" iyz="0.00" izz="${Jz}"/>
     </inertial>
     <visual name="plane_visual">
-      <origin xyz="0 0 0" rpy="0 0 1.570796" />
+      <origin xyz="0 0 0" rpy="0 0 1.570796"/>
       <geometry>
-        <mesh filename="${mesh_file}">
-          <submesh name="Wing" center="true" />
-        </mesh>
+        <!-- <mesh filename="${mesh_file}"> <submesh name="Wing" center="true" /> </mesh> -->
+        <box size="${body_width} ${body_height} ${body_length}"/>
       </geometry>
     </visual>
     <collision name="plane_collision">
-      <origin xyz="0 0 0" rpy="0 0 1.570796" />
+      <origin xyz="0 0 0" rpy="0 0 1.570796"/>
       <geometry>
-        <box size="${body_width} ${body_height} ${body_length}" />
+        <box size="${body_width} ${body_height} ${body_length}"/>
       </geometry>
     </collision>
   </link>
+  <gazebo reference="${namespace}/base_link">
+    <collision name="plane_collision">
+      <surface>
+        <friction>
+          <ode>
+            <mu>0.01</mu>
+            <mu2>0.01</mu2>
+          </ode>
+        </friction>
+      </surface>
+    </collision>
+  </gazebo>
   <!-- Simulator Truth -->
   <xacro:include filename="$(find rosplane_sim)/xacro/aircraft_truth.xacro"/>
-  <xacro:aircraft_truth
-    namespace="${namespace}"
-    parent_link="${namespace}/base_link"/>
+  <xacro:aircraft_truth namespace="${namespace}" parent_link="${namespace}/base_link"/>
   <!-- Aerodynamics -->
   <xacro:include filename="$(find rosplane_sim)/xacro/aircraft_forces_and_moments.xacro"/>
-  <xacro:aircraft_dynamics
-    namespace="${namespace}"
-    parent_link="${namespace}/base_link"/>
+  <xacro:aircraft_dynamics namespace="${namespace}" parent_link="${namespace}/base_link"/>
   <!-- GPS -->
   <xacro:include filename="$(find rosflight_plugins)/xacro/GPS.xacro"/>
-  <xacro:gps_plugin_macro
-    namespace="${namespace}"
-    parent_link="${namespace}/base_link">
-  </xacro:gps_plugin_macro>
+  <xacro:gps_plugin_macro namespace="${namespace}" parent_link="${namespace}/base_link"></xacro:gps_plugin_macro>
   <!-- IMU -->
   <xacro:include filename="$(find rosflight_plugins)/xacro/imu.xacro"/>
-  <xacro:imu_plugin_macro
-    namespace="${namespace}"
-    parent_link="${namespace}/base_link">
-  </xacro:imu_plugin_macro>
+  <xacro:imu_plugin_macro namespace="${namespace}" parent_link="${namespace}/base_link"></xacro:imu_plugin_macro>
   <!-- Airspeed -->
   <xacro:include filename="$(find rosflight_plugins)/xacro/airspeed.xacro"/>
-  <xacro:airspeed_plugin_macro
-    namespace="${namespace}"
-    parent_link="${namespace}/base_link">
-  </xacro:airspeed_plugin_macro>
+  <xacro:airspeed_plugin_macro namespace="${namespace}" parent_link="${namespace}/base_link"></xacro:airspeed_plugin_macro>
   <!-- Barometer -->
   <xacro:include filename="$(find rosflight_plugins)/xacro/barometer.xacro"/>
-  <xacro:barometer_plugin_macro
-    namespace="${namespace}"
-    parent_link="${namespace}/base_link">
-  </xacro:barometer_plugin_macro>
+  <xacro:barometer_plugin_macro namespace="${namespace}" parent_link="${namespace}/base_link"></xacro:barometer_plugin_macro>
   <!-- Chase Camera -->
-  <!-- <xacro:include filename="$(find magicc_sim_plugins)/xacro/camera.xacro"/>
-  <xacro:simple_camera
-    namespace="${namespace}/chase"
-    frame_rate="30"
-    rgb_range="1000"
-    parent_link="${namespace}/base_link"
-    image_topic="rgb"
-    image_camera_info_topic="camera_info">
-    <origin xyz="-${1.1*body_length} 0 ${0.8*body_height}"/>
-  </xacro:simple_camera> -->
+  <!-- <xacro:include filename="$(find magicc_sim_plugins)/xacro/camera.xacro"/> <xacro:simple_camera namespace="${namespace}/chase" frame_rate="30" rgb_range="1000" parent_link="${namespace}/base_link" image_topic="rgb"
+  image_camera_info_topic="camera_info"> <origin xyz="-${1.1*body_length} 0 ${0.8*body_height}"/> </xacro:simple_camera> -->
   <!-- Gimbal -->
-  <!-- <xacro:include filename="$(find magicc_sim_plugins)/xacro/gimbal.xacro"/>
-  <xacro:gimbal_ZENMUSE
-    namespace="${namespace}"
-    parent_link="${namespace}/base_link"
-    camera_topic="rgb"
-    frame_rate="30"
-    pose_topic="${namespace}/gimbal/pose"
-    command_topic="${namespace}/gimbal/control"
-    use_slipring="true">
-    <origin xyz="-${0.4*body_length} 0 -${0.4*body_height}" rpy="0 0 0"/>
-  </xacro:gimbal_ZENMUSE> -->
+  <!-- <xacro:include filename="$(find magicc_sim_plugins)/xacro/gimbal.xacro"/> <xacro:gimbal_ZENMUSE namespace="${namespace}" parent_link="${namespace}/base_link" camera_topic="rgb" frame_rate="30" pose_topic="${namespace}/gimbal/pose"
+  command_topic="${namespace}/gimbal/control" use_slipring="true"> <origin xyz="-${0.4*body_length} 0 -${0.4*body_height}" rpy="0 0 0"/> </xacro:gimbal_ZENMUSE> -->
 </robot>
